File: hw/zvonecek/primary.kicad_sch (KiCad schematic)
At the start: 35 parts, among them J1 Conn_01x06_Male, J2 01x06, SW1 SW_SPST, SW10 SW_SPST, SW11 SW_SPST, SW12 SW_SPST, SW13 SW_SPST, SW14 SW_DP3T, SW2 SW_SPST, SW3 SW_SPST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

Commit message: HW design 1.0 as manufactured
Signed-off-by: Jan Hamal Dvořák <mordae@anilinux.org>
Parts:
- removed J2: 01x06, Connector_PinHeader_2.54mm:PinHeader_1x06_P2.54mm_Horizontal, symbol Connector_Generic:Conn_01x06
- removed LS1: Speaker, Connector_PinHeader_2.54mm:PinHeader_1x02_P2.54mm_Horizontal, symbol Device:Speaker
- added C3: 22u, Capacitor_SMD:C_0603_1608Metric, symbol Device:C
- added J10, J9: Conn_01x02_Male, Connector_PinHeader_2.54mm:PinHeader_1x02_P2.54mm_Vertical, symbol Connector:Conn_01x02_Male
- added J4: 01x02, Connector_PinHeader_2.54mm:PinHeader_1x02_P2.54mm_Vertical, symbol Connector:Conn_01x02_Male
- added J5, J8: Conn_01x01_Male, Connector_PinHeader_2.54mm:PinHeader_1x01_P2.54mm_Vertical, symbol Connector:Conn_01x01_Male
- J1: footprint Connector_PinHeader_2.54mm:PinHeader_1x06_P2.54mm_Horizontal -> Connector_PinHeader_2.54mm:PinHeader_1x06_P2.54mm_Vertical
- R1, R2, R3: footprint Resistor_THT:R_Axial_DIN0204_L3.6mm_D1.6mm_P5.08mm_Horizontal -> Resistor_SMD:R_0603_1608Metric
- U1: footprint RF_Module:ESP32-WROOM-32 -> Library:ESP32-WROOM-32
Connections:
- net +3V3: now also C3.2, J9.1 (Pin_1)
- net +BATT: now also J4.1 (Pin_1)
- net BOOT: now also J8.1 (Pin_1)
- net EN: now also J5.1 (Pin_1)
- net GND: now also C3.1, J4.2 (Pin_2), J9.2 (Pin_2)
- net I2S-BCLK: now also U1.9 (IO33); no longer U1.12 (IO27)
- net I2S-DATA: now also U1.10 (IO25); no longer U1.8 (IO32)
- net I2S-WS: now also U1.8 (IO32); no longer U1.9 (IO33)
- net KEY1: now also U1.12 (IO27); no longer U1.31 (IO19)
- net KEY2: now also U1.13 (IO14); no longer U1.33 (IO21)
- net KEY3: now also U1.14 (IO12); no longer U1.36 (IO22)
- net KEY4: now also U1.16 (IO13); no longer U1.37 (IO23)
- net KEY5: now also U1.23 (IO15); no longer U1.10 (IO25)
- net KEY6: now also U1.24 (IO2); no longer U1.11 (IO26)
- net LED: now also U1.27 (IO16); no longer U1.24 (IO2)
- net ROW1: now also U1.11 (IO26); no longer U1.27 (IO16)
- net ROW2: now also U1.26 (IO4); no longer U1.28 (IO17)
- net ROW3: now also U1.28 (IO17); no longer U1.30 (IO18)
- net RX: now also J10.2 (Pin_2)
- net SD-CS: now also U1.37 (IO23); no longer U1.23 (IO15)
- net SD-MISO: now also U1.31 (IO19); no longer U1.14 (IO12)
- net SD-MOSI: now also U1.36 (IO22); no longer U1.16 (IO13)
- net SD-SCLK: now also U1.33 (IO21); no longer U1.13 (IO14)
- net TX: now also J10.1 (Pin_1)
- net VOL: now also U1.30 (IO18); no longer U1.26 (IO4)
Other:
- moved on the sheet: BT1, C1
