File: hw/zvonecek/secondary.kicad_sch (KiCad schematic)
At the start: 6 parts, among them J3 Conn_01x06_Male, SW15 SW_SPST, SW16 SW_SPST, SW17 SW_SPST, SW18 SW_SPST, SW19 SW_SPST

Commit message: HW design 1.0 as manufactured
Signed-off-by: Jan Hamal Dvořák <mordae@anilinux.org>
Parts:
- J3: footprint Connector_PinHeader_2.54mm:PinHeader_1x06_P2.54mm_Horizontal -> Connector_PinHeader_2.54mm:PinHeader_1x06_P2.54mm_Vertical
- SW15: footprint Library:BUTTON-RA -> Library:BUTTON
- SW16: footprint Library:BUTTON-RA-ALT -> Library:BUTTON
