File: hw/zvonecek/zvonecek.kicad_pcb (KiCad board)
At the start: 2 copper layers, 199.4 x 92.5 mm, 40 parts, among them J1 Conn_01x06_Male, J2 01x06, J3 Conn_01x06_Male, SW1 SW_SPST, SW10 SW_SPST, SW11 SW_SPST, SW12 SW_SPST, SW13 SW_SPST, SW14 SW_DP3T, SW15 SW_SPST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

Commit message: HW design 1.0 as manufactured
Signed-off-by: Jan Hamal Dvořák <mordae@anilinux.org>
Parts:
- removed J2: 01x06, Connector_PinHeader_2.54mm:PinHeader_1x06_P2.54mm_Horizontal
- removed LS1: Speaker, Connector_PinHeader_2.54mm:PinHeader_1x02_P2.54mm_Horizontal
- added C3: 22u, Capacitor_SMD:C_0603_1608Metric, F.Cu at (115.8, 79.9)
- added J10: Conn_01x02_Male, Connector_PinHeader_2.54mm:PinHeader_1x02_P2.54mm_Vertical, B.Cu at (146.5, 82.5)
- added J4: 01x02, Connector_PinHeader_2.54mm:PinHeader_1x02_P2.54mm_Vertical, B.Cu at (231.6, 79.9)
- added J5: Conn_01x01_Male, Connector_PinHeader_2.54mm:PinHeader_1x01_P2.54mm_Vertical, B.Cu at (112.2, 85.1)
- added J8: Conn_01x01_Male, Connector_PinHeader_2.54mm:PinHeader_1x01_P2.54mm_Vertical, B.Cu at (137.6, 100.3)
- added J9: Conn_01x02_Male, Connector_PinHeader_2.54mm:PinHeader_1x02_P2.54mm_Vertical, B.Cu at (65.9, 83.2)
- J1: footprint Connector_PinHeader_2.54mm:PinHeader_1x06_P2.54mm_Horizontal -> Connector_PinHeader_2.54mm:PinHeader_1x06_P2.54mm_Vertical
- J3: footprint Connector_PinHeader_2.54mm:PinHeader_1x06_P2.54mm_Horizontal -> Connector_PinHeader_2.54mm:PinHeader_1x06_P2.54mm_Vertical; moved to F.Cu
- R1, R2, R3: footprint Resistor_THT:R_Axial_DIN0204_L3.6mm_D1.6mm_P5.08mm_Horizontal -> Resistor_SMD:R_0603_1608Metric
- SW15: footprint Library:BUTTON-RA -> Library:BUTTON
- SW16: footprint Library:BUTTON-RA-ALT -> Library:BUTTON
- U1: footprint RF_Module:ESP32-WROOM-32 -> Library:ESP32-WROOM-32
- U2, U3, U4: moved to B.Cu
- moved U2 338.7 mm to (221.4, 95.2), turned to -90 degrees
- moved SW14 336.2 mm to (244.5, 88.0), turned to -10 degrees
- moved SW12 295.3 mm to (212.5, 119.5), turned to 90 degrees
- moved U3 293.6 mm to (202.4, 76.2), turned to 90 degrees
- moved D8 284.2 mm to (236.5, 106.2), turned to 180 degrees
- moved SW13 279.4 mm to (236.4, 113.6), turned to 90 degrees
- moved D7 277.7 mm to (212.6, 112.0), turned to 180 degrees
- moved SW11 249.5 mm to (188.8, 122.5), turned to 90 degrees
- moved U1 245.9 mm to (129.4, 87.7)
- moved D6 245.4 mm to (188.5, 115.2), turned to 180 degrees
- moved R1 235.2 mm to (113.4, 81.5), turned to -90 degrees
- moved R2 226.2 mm to (96.3, 81.5), turned to -90 degrees
- moved C1 222.8 mm to (117.3, 79.9), turned to -90 degrees
- moved R3 212.8 mm to (98.9, 81.5), turned to 90 degrees
- moved D5 210.2 mm to (164.4, 117.1), turned to 180 degrees
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Connections:
- U1 pad 10: KEY5 -> I2S-DATA
- U1 pad 11: KEY6 -> ROW1
- U1 pad 12: I2S-BCLK -> KEY1
- U1 pad 13: SD-SCLK -> KEY2
- U1 pad 14: SD-MISO -> KEY3
- U1 pad 16: SD-MOSI -> KEY4
- U1 pad 23: SD-CS -> KEY5
- U1 pad 24: LED -> KEY6
- U1 pad 26: VOL -> ROW2
- U1 pad 27: ROW1 -> LED
- U1 pad 28: ROW2 -> ROW3
- U1 pad 30: ROW3 -> VOL
- U1 pad 31: KEY1 -> SD-MISO
- U1 pad 33: KEY2 -> SD-SCLK
- U1 pad 36: KEY3 -> SD-MOSI
- U1 pad 37: KEY4 -> SD-CS
- U1 pad 8: I2S-DATA -> I2S-WS
- U1 pad 9: I2S-WS -> I2S-BCLK
Routing:
- net +3V3: track 0.00 -> 400.9 mm, vias 0 -> 18
- net ROW2: track 0.00 -> 201.0 mm, vias 0 -> 7
- net KEY6: track 0.00 -> 192.3 mm, vias 0 -> 4
- net ROW3: track 0.00 -> 182.0 mm, vias 0 -> 4
- net KEY5: track 104.5 -> 276.4 mm, vias 0 -> 8
- net KEY4: track 75.8 -> 241.1 mm, vias 0 -> 5
- net KEY3: track 47.7 -> 196.8 mm, vias 0 -> 6
- net KEY2: track 9.30 -> 154.6 mm, vias 0 -> 4
- net VOL: track 0.00 -> 116.2 mm
- net KEY1: track 19.4 -> 121.1 mm, vias 0 -> 2
- net ROW1: track 138.0 -> 56.1 mm
- net LED: track 0.00 -> 79.5 mm, vias 0 -> 2
- net SD-CS: track 0.00 -> 70.2 mm
- net SD-SCLK: track 0.00 -> 68.8 mm
- net SD-MOSI: track 0.00 -> 67.9 mm
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- added copper zone on B.Cu, net GND
- added copper zone on F.Cu, net GND
- added copper zone on B.Cu, net ROW1
Other:
- board size 199.4 x 92.5 mm -> 200 x 80.3 mm
- board text added: "Desku ve spěchu navrhoval: Strejda Mordae"
- board text added: "Jankolovi & Hamalovi"
- board text added: "Nástroj hrůzy a zmaru"
- board text added: "Vyroben pro Violku v roce 2022 v Praze"
- board text added: "Zvoneček 1.0"
